Commit message: Colors added

File: arm_description/urdf/arm.urdf.xacro (robot description, xacro)
@@ -24,9 +24,19 @@
   <xacro:property name="base_mass"   value="1.0"/>
   <xacro:property name="link_mass"   value="0.3"/>
+  <xacro:property name="sphere_mass" value="0.1"/>
   <xacro:property name="hand_mass"   value="0.1"/>
   <xacro:property name="finger_mass" value="0.05"/>
-  <!-- ===== MATERIALS ===== -->
+  <!-- Gazebo colors -->
+  <xacro:property name="arm_color"    value="Gazebo/Orange"/>
+  <xacro:property name="joint_color"  value="Gazebo/Black"/>
+  <xacro:property name="base_color"   value="Gazebo/DarkGrey"/>
+  <xacro:property name="hand_color"   value="Gazebo/Black"/>
+  <xacro:property name="finger_color" value="Gazebo/White"/>
+  <!-- ===== MATERIALS (RViz colors) ===== -->
   <material name="black">
     <color rgba="0 0 0 1"/>
+  </material>
+  <material name="orange">
+    <color rgba="1 0.5 0 1"/>
   </material>
   <material name="white">
@@ -61,5 +71,5 @@
     </inertial>
   </xacro:macro>
-  <!-- ===== ARM SEGMENT MACRO: cylinder, optional top sphere, and its revolute joint ===== -->
+  <!-- ===== ARM SEGMENT MACRO: cylinder link, its revolute joint, and an optional joint sphere on top ===== -->
   <xacro:macro name="arm_segment" params="index parent joint_z top_sphere axis">
     <link name="link${index}">
@@ -69,5 +79,5 @@
         </geometry>
         <origin xyz="0 0 ${segment_length/2}" rpy="0 0 0"/>
-        <material name="white"/>
+        <material name="orange"/>
       </visual>
       <collision>
@@ -77,19 +87,4 @@
         <origin xyz="0 0 ${segment_length/2}" rpy="0 0 0"/>
       </collision>
-      <xacro:if value="${top_sphere}">
-        <visual>
-          <geometry>
-            <sphere radius="${joint_radius}"/>
-          </geometry>
-          <origin xyz="0 0 ${segment_length}" rpy="0 0 0"/>
-          <material name="black"/>
-        </visual>
-        <collision>
-          <geometry>
-            <sphere radius="${joint_radius}"/>
-          </geometry>
-          <origin xyz="0 0 ${segment_length}" rpy="0 0 0"/>
-        </collision>
-      </xacro:if>
       <xacro:inertial_cylinder mass="${link_mass}" r="${link_radius}" h="${link_length}" xyz="0 0 ${segment_length/2}"/>
     </link>
@@ -101,4 +96,35 @@
       <limit lower="${-joint_limit}" upper="${joint_limit}" effort="${joint_effort}" velocity="${joint_velocity}"/>
     </joint>
+    <gazebo reference="link${index}">
+      <material>${arm_color}</material>
+    </gazebo>
+    <!-- Joint sphere: separate link so it can have its own color -->
+    <xacro:if value="${top_sphere}">
+      <link name="link${index}_sphere">
+        <visual>
+          <geometry>
+            <sphere radius="${joint_radius}"/>
+          </geometry>
+          <material name="black"/>
+        </visual>
+        <collision>
+          <geometry>
+            <sphere radius="${joint_radius}"/>
+          </geometry>
+        </collision>
+        <xacro:inertial_sphere mass="${sphere_mass}" r="${joint_radius}" xyz="0 0 0"/>
+      </link>
+      <joint name="link${index}_to_sphere" type="fixed">
+        <parent link="link${index}"/>
+        <child link="link${index}_sphere"/>
+        <origin xyz="0 0 ${segment_length}" rpy="0 0 0"/>
+      </joint>
+      <gazebo reference="link${index}_sphere">
+        <material>${joint_color}</material>
+      </gazebo>
+      <gazebo reference="link${index}_to_sphere">
+        <preserveFixedJoint>true</preserveFixedJoint>
+      </gazebo>
+    </xacro:if>
   </xacro:macro>
   <!-- ===== FINGER MACRO. reflect = 1 for left, -1 for right ===== -->
@@ -127,4 +153,7 @@
       <limit lower="0" upper="${finger_travel}" effort="${joint_effort}" velocity="${joint_velocity}"/>
     </joint>
+    <gazebo reference="gripper_finger_${side}">
+      <material>${finger_color}</material>
+    </gazebo>
   </xacro:macro>
   <!-- ===== ROS 2 CONTROL JOINT MACRO ===== -->
@@ -153,5 +182,8 @@
     <xacro:inertial_sphere mass="${base_mass}" r="${joint_radius}" xyz="0 0 0"/>
   </link>
-  <!-- Lifted by the sphere's radius so the base sits on the ground instead of half inside it -->
+  <gazebo reference="base_link">
+    <material>${base_color}</material>
+  </gazebo>
+  <!-- Lifted by the sphere's radius so the base sits on the ground -->
   <joint name="world_to_base" type="fixed">
     <parent link="world"/>
@@ -178,4 +210,7 @@
     <xacro:inertial_box mass="${hand_mass}" x="${hand_x}" y="${hand_y}" z="${hand_z}" xyz="0 0 ${hand_z/2}"/>
   </link>
+  <gazebo reference="gripper_hand">
+    <material>${hand_color}</material>
+  </gazebo>
   <joint name="gripper_joint" type="fixed">
     <parent link="link3"/>

Commit message: Version 2: IK-based reach control and visual update
- Reach controlled by hand distance from camera, using inverse kinematics
- Calibrated hand-size range for reach
- Gazebo colors with separate black joint links
- Gripper back to position control for smooth motion
- Removed pick-and-place world

File: arm_description/urdf/arm.urdf.xacro (robot description, xacro)
@@ -21,4 +21,5 @@
   <xacro:property name="finger_height"   value="0.07"/>
   <xacro:property name="finger_travel"   value="0.027"/>
+  <xacro:property name="finger_effort"   value="5"/>     <!-- max finger force in N -->
   <!-- Masses (kg) -->
   <xacro:property name="base_mass"   value="1.0"/>
@@ -123,4 +124,5 @@
         <material>${joint_color}</material>
       </gazebo>
+      <!-- Stop Gazebo from merging the sphere into its parent link (keeps its color) -->
       <gazebo reference="link${index}_to_sphere">
         <preserveFixedJoint>true</preserveFixedJoint>
@@ -151,6 +153,7 @@
       <origin xyz="0 0 0" rpy="0 0 0"/>
       <axis xyz="0 ${-reflect} 0"/>
-      <limit lower="0" upper="${finger_travel}" effort="${joint_effort}" velocity="${joint_velocity}"/>
-    </joint>
+      <limit lower="0" upper="${finger_travel}" effort="${finger_effort}" velocity="${joint_velocity}"/>
+    </joint>
+    <!-- Color and high-friction contact, so the fingers can grip -->
     <gazebo reference="gripper_finger_${side}">
       <material>${finger_color}</material>
@@ -163,8 +166,17 @@
     </gazebo>
   </xacro:macro>
-  <!-- ===== ROS 2 CONTROL JOINT MACRO ===== -->
+  <!-- ===== ROS 2 CONTROL JOINT MACROS ===== -->
+  <!-- Position-controlled joint (arm) -->
   <xacro:macro name="control_joint" params="name">
     <joint name="${name}">
       <command_interface name="position"/>
+      <state_interface name="position"/>
+      <state_interface name="velocity"/>
+    </joint>
+  </xacro:macro>
+  <!-- Effort-controlled joint (gripper fingers): limited force, stops on contact -->
+  <xacro:macro name="control_joint_effort" params="name">
+    <joint name="${name}">
+      <command_interface name="effort"/>
       <state_interface name="position"/>
       <state_interface name="velocity"/>

Commit message: Updated to Jazzy

File: arm_description/urdf/arm.urdf.xacro (robot description, xacro)
@@ -21,5 +21,4 @@
   <xacro:property name="finger_height"   value="0.07"/>
   <xacro:property name="finger_travel"   value="0.027"/>
-  <xacro:property name="finger_effort"   value="5"/>     <!-- max finger force in N -->
   <!-- Masses (kg) -->
   <xacro:property name="base_mass"   value="1.0"/>
@@ -28,13 +27,7 @@
   <xacro:property name="hand_mass"   value="0.1"/>
   <xacro:property name="finger_mass" value="0.05"/>
-  <!-- Gazebo colors -->
-  <xacro:property name="arm_color"    value="Gazebo/Orange"/>
-  <xacro:property name="joint_color"  value="Gazebo/Black"/>
-  <xacro:property name="base_color"   value="Gazebo/DarkGrey"/>
-  <xacro:property name="hand_color"   value="Gazebo/Black"/>
-  <xacro:property name="finger_color" value="Gazebo/White"/>
-  <!-- ===== MATERIALS (RViz colors) ===== -->
+  <!-- ===== MATERIALS (used by both RViz and the new Gazebo) ===== -->
   <material name="black">
-    <color rgba="0 0 0 1"/>
+    <color rgba="0.05 0.05 0.05 1"/>
   </material>
   <material name="orange">
@@ -97,8 +90,5 @@
       <limit lower="${-joint_limit}" upper="${joint_limit}" effort="${joint_effort}" velocity="${joint_velocity}"/>
     </joint>
-    <gazebo reference="link${index}">
-      <material>${arm_color}</material>
-    </gazebo>
-    <!-- Joint sphere: separate link so it can have its own color -->
+    <!-- Joint sphere -->
     <xacro:if value="${top_sphere}">
       <link name="link${index}_sphere">
@@ -121,11 +111,4 @@
         <origin xyz="0 0 ${segment_length}" rpy="0 0 0"/>
       </joint>
-      <gazebo reference="link${index}_sphere">
-        <material>${joint_color}</material>
-      </gazebo>
-      <!-- Stop Gazebo from merging the sphere into its parent link (keeps its color) -->
-      <gazebo reference="link${index}_to_sphere">
-        <preserveFixedJoint>true</preserveFixedJoint>
-      </gazebo>
     </xacro:if>
   </xacro:macro>
@@ -153,19 +136,8 @@
       <origin xyz="0 0 0" rpy="0 0 0"/>
       <axis xyz="0 ${-reflect} 0"/>
-      <limit lower="0" upper="${finger_travel}" effort="${finger_effort}" velocity="${joint_velocity}"/>
+      <limit lower="0" upper="${finger_travel}" effort="${joint_effort}" velocity="${joint_velocity}"/>
     </joint>
-    <!-- Color and high-friction contact, so the fingers can grip -->
-    <gazebo reference="gripper_finger_${side}">
-      <material>${finger_color}</material>
-      <mu1>2.0</mu1>
-      <mu2>2.0</mu2>
-      <kp>1000000.0</kp>
-      <kd>100.0</kd>
-      <minDepth>0.001</minDepth>
-      <maxVel>0.1</maxVel>
-    </gazebo>
-  </xacro:macro>
-  <!-- ===== ROS 2 CONTROL JOINT MACROS ===== -->
-  <!-- Position-controlled joint (arm) -->
+  </xacro:macro>
+  <!-- ===== ROS 2 CONTROL JOINT MACRO ===== -->
   <xacro:macro name="control_joint" params="name">
     <joint name="${name}">
@@ -175,12 +147,4 @@
     </joint>
   </xacro:macro>
-  <!-- Effort-controlled joint (gripper fingers): limited force, stops on contact -->
-  <xacro:macro name="control_joint_effort" params="name">
-    <joint name="${name}">
-      <command_interface name="effort"/>
-      <state_interface name="position"/>
-      <state_interface name="velocity"/>
-    </joint>
-  </xacro:macro>
   <!-- ===== ROBOT ===== -->
   <!-- World: pins the arm to the ground in Gazebo -->
@@ -200,7 +164,4 @@
     <xacro:inertial_sphere mass="${base_mass}" r="${joint_radius}" xyz="0 0 0"/>
   </link>
-  <gazebo reference="base_link">
-    <material>${base_color}</material>
-  </gazebo>
   <!-- Lifted by the sphere's radius so the base sits on the ground -->
   <joint name="world_to_base" type="fixed">
@@ -228,7 +189,4 @@
     <xacro:inertial_box mass="${hand_mass}" x="${hand_x}" y="${hand_y}" z="${hand_z}" xyz="0 0 ${hand_z/2}"/>
   </link>
-  <gazebo reference="gripper_hand">
-    <material>${hand_color}</material>
-  </gazebo>
   <joint name="gripper_joint" type="fixed">
     <parent link="link3"/>
@@ -238,8 +196,8 @@
   <xacro:finger side="left"  reflect="1"/>
   <xacro:finger side="right" reflect="-1"/>
-  <!-- ===== ROS 2 CONTROL ===== -->
-  <ros2_control name="GazeboSystem" type="system">
+  <!-- ===== ROS 2 CONTROL (new Gazebo) ===== -->
+  <ros2_control name="GazeboSimSystem" type="system">
     <hardware>
-      <plugin>gazebo_ros2_control/GazeboSystem</plugin>
+      <plugin>gz_ros2_control/GazeboSimSystem</plugin>
     </hardware>
     <xacro:control_joint name="joint1"/>
@@ -250,5 +208,5 @@
   </ros2_control>
   <gazebo>
-    <plugin filename="libgazebo_ros2_control.so" name="gazebo_ros2_control">
+    <plugin filename="gz_ros2_control-system" name="gz_ros2_control::GazeboSimROS2ControlPlugin">
       <parameters>$(find arm_description)/config/arm_controllers.yaml</parameters>
     </plugin>
